File: kicad/simple-incubator/simple-incubator.kicad_pcb (KiCad board)
At the start: 2 copper layers, 16 parts, among them J1 Conn_Coaxial_Power, J2 Fan, J3 Onewire1, J4 FT232L, J5 Onewire2, Q1 BSP75, Q2 IRF3704, SW1 Rotary_Encoder_Switch, U1 MCP1703A-5002_SOT223, U2 ATmega328-AU

Commit message: update kicad
Parts:
- added R2: R, Resistor_SMD:R_0805_2012Metric_Pad1.15x1.40mm_HandSolder, B.Cu at (305.3, 151.7)
- C1, C2, C3, J1, J2, J3, J4, J5, Q2, R1, SP1, U1: moved to B.Cu
- moved Q1 148.1 mm to (47.2, 73.2)
- moved SP1 125.2 mm to (259.5, 111.3)
- moved J4 125.1 mm to (235.6, 131.9)
- moved J5 125.1 mm to (267.9, 131.9)
- moved J2 124.7 mm to (264.1, 130.5)
- moved J1 124.1 mm to (305.0, 128.3)
- moved C2 124.0 mm to (244.3, 127.5)
- moved R1 124.0 mm to (248.1, 127.5)
- moved Q2 123.6 mm to (268.9, 125.1)
- moved J3 123.6 mm to (235.6, 125.0)
- moved C3 123.5 mm to (278.5, 123.7)
- moved C1 123.5 mm to (244.3, 122.7)
- moved U1 119.3 mm to (255.8, 185.2)
- moved SW1 110.8 mm to (278.9, 155.4)
- moved DS1 103.7 mm to (216.9, 107.7)
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Connections:
- net Net-(SP1-Pad1) renamed /LCD_MISO
- net Net-(SP1-Pad4) renamed /LCD2_MOS1
- net Net-(SP1-Pad5) renamed /RESET
- net Net-(U2-Pad2) renamed /D4
- net Net-(U2-Pad9) renamed /PD5
- DS1 pad 11: Net-(DS1-Pad11) -> /LCD1
- DS1 pad 12: Net-(DS1-Pad12) -> /LCD2_MOSI
- DS1 pad 13: Net-(DS1-Pad13) -> /LCD3_MISO
- DS1 pad 14: Net-(DS1-Pad14) -> /LCD4_SCK
- DS1 pad 16: Net-(DS1-Pad16) -> GND
- DS1 pad 2: +5V -> VCC
- DS1 pad 3: Net-(DS1-Pad3) -> VCC
- DS1 pad 4: Net-(DS1-Pad4) -> /LCD_RS
- DS1 pad 5: Net-(DS1-Pad5) -> /LCD_RW
- DS1 pad 6: Net-(DS1-Pad6) -> /LCD_E
- SP1 pad 3: Net-(SP1-Pad3) -> /LCD4_SCK
- SP1 pad 6: Net-(SP1-Pad6) -> GND
- SW1 pad A: Net-(SW1-PadA) -> /D3
- SW1 pad B: Net-(SW1-PadB) -> /D2
- SW1 pad C: Net-(SW1-PadC) -> GND
- SW1 pad S1: Net-(SW1-PadS1) -> GND
- U2 pad 1: Net-(U2-Pad1) -> /D3
- U2 pad 10: Net-(U2-Pad10) -> /LCD_RS
- U2 pad 11: Net-(U2-Pad11) -> /LCD_RW
- U2 pad 12: Net-(U2-Pad12) -> /LCD_E
- U2 pad 13: Net-(U2-Pad13) -> /LCD_LED
- U2 pad 14: Net-(U2-Pad14) -> /LCD1
- U2 pad 15: Net-(U2-Pad15) -> /LCD2_MOSI
- U2 pad 16: Net-(U2-Pad16) -> /LCD3_MISO
- U2 pad 17: Net-(U2-Pad17) -> /LCD4_SCK
- U2 pad 32: Net-(U2-Pad32) -> /D2
Routing:
- net /D2: track 0.00 -> 78.0 mm
- net GND: track 0.00 -> 5.05 mm
Other:
- board outline added: 288.8 x 188.8 mm

Commit message: The footprint should have changed to simple footprint design with 9 pads and a hole.
Parts:
- removed C1, C2, C3: C, Capacitor_SMD:C_0805_2012Metric_Pad1.15x1.40mm_HandSolder
- removed DS1: WC1602A, Display:WC1602A
- removed J1: Conn_Coaxial_Power, Connector_BarrelJack:BarrelJack_Horizontal
- removed J2: Fan, Connector_BarrelJack:BarrelJack_Horizontal
- removed J3: Onewire1, Connector_Molex:Molex_KK-254_AE-6410-03A_1x03_P2.54mm_Vertical
- removed J4: FT232L, Connector_Molex:Molex_KK-254_AE-6410-06A_1x06_P2.54mm_Vertical
- removed J5: Onewire2, Connector_Molex:Molex_KK-254_AE-6410-04A_1x04_P2.54mm_Vertical
- removed Q1: BSP75, Package_TO_SOT_SMD:SOT-223-3_TabPin2
- removed Q2: IRF3704, Package_TO_SOT_THT:TO-220-3_Vertical
- removed R1: 10k, Resistor_SMD:R_0805_2012Metric_Pad1.15x1.40mm_HandSolder
- removed R2: R, Resistor_SMD:R_0805_2012Metric_Pad1.15x1.40mm_HandSolder
- removed SP1: ICSP, Connector:Tag-Connect_TC2030-IDC-NL_2x03_P1.27mm_Vertical
- removed SW1: Rotary_Encoder_Switch, Rotary_Encoder:RotaryEncoder_Alps_EC11E-Switch_Vertical_H20mm
- removed U1: MCP1703A-5002_SOT223, Package_TO_SOT_SMD:SOT-223-3_TabPin2
- removed U2: ATmega328-AU, Package_QFP:TQFP-32_7x7mm_P0.8mm
Routing:
- net /D2: track 78.0 -> 0.00 mm
- net GND: track 5.05 -> 0.00 mm
Other:
- outline, holes or cut-outs redrawn
