File: kicad/simple-incubator/_autosave-simple-incubator.kicad_pcb (KiCad board)
At the start: 2 copper layers, 288.8 x 188.8 mm, 8 parts, among them J1 Conn_Coaxial_Power, J2 RJ12, J3 Onewire1, J5 Onewire2, Q1 BSP75, U1 MCP1703A-5002_SOT223

Commit message: last weeks updates
Parts:
- moved J2 9.18 mm to (205.7, 130.8)
Changed lines of the file:
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@@
   )
   (module Connector_RJ:RJ12_Amphenol_54601 (layer F.Cu)
-    (at 214.885001 130.025001)
+    (at 205.74 130.81)
     (descr "RJ12 connector  https://cdn.amphenol-icc.com/media/wysiwyg/files/drawing/c-bmj-0082.pdf")
     (tags "RJ12 connector")
