File: Kicad/incubator_bottom/incubator_bottom.sch (KiCad schematic (older format))
At the start: 29 parts, among them J1 Conn_01x02, J2 Conn_02x03_Odd_Even, J3 RJ12, J4 Conn_01x05, J5 AudioJack3_SwitchTR, J6 AudioJack3_SwitchTR, Q1 ZXMS6004, U1 DS18B20Z, U2 DS18B20

Commit message: refactor: Kicad design updated
Parts:
- added C3, C4, C5: 100n, Capacitor_SMD:C_0805_2012Metric_Pad1.18x1.45mm_HandSolder, symbol Device:C
- added D2: MBR0520LT, Diode_SMD:D_SOD-123, symbol Diode:MBR0520LT
- added J7: Conn_01x02, Connector_JST:JST_XH_B2B-XH-A_1x02_P2.50mm_Vertical, symbol Connector_Generic:Conn_01x02
- added J8: Conn_01x06, Connector_PinHeader_2.54mm:PinHeader_1x06_P2.54mm_Vertical, symbol Connector_Generic:Conn_01x06
- added Q2: IPB80N03S4L-03, Package_TO_SOT_SMD:TO-263-2, symbol Bertha_main:IPB80N03S4L-03
- added R13: 100, Resistor_SMD:R_0805_2012Metric_Pad1.20x1.40mm_HandSolder, symbol Device:R
- H5, H6, H7, H8: footprint MountingHole:MountingHole_3.2mm_M3 -> MountingHole:MountingHole_4.3mm_M4
- J1: footprint Connector_JST:JST_EH_B2B-EH-A_1x02_P2.50mm_Vertical -> Connector_JST:JST_XH_B2B-XH-A_1x02_P2.50mm_Vertical
Connections:
- net +12V: now also J4.1 (Pin_1), J7.2 (Pin_2)
- net GND: now also C3.2, C4.2, C5.2, J8.6 (Pin_6), Q2.3 (S)
- net VIN: now also D2.1 (K)
- net ~RESET: now also C5.1, J8.1 (Pin_1)
- net FAN: now reaches Q1.1 (G)
- net FAN: now also C3.1
- new net: J7.1 (Pin_1), Q2.2 (D)
- new net: C4.1, Q2.1 (G), R13.1
- new net: D2.2 (A), J8.4 (Pin_4)
- new net PID: R13.2
- new net RX: J8.3 (Pin_3)
- new net TX: J8.2 (Pin_2)
- no-connect marks 7 -> 8
Other:
- moved on the sheet: J1, Q1

Commit message: refactor: Kicad design updated
Other:
- note added: "PID"
Changed lines of the file:
@@
 Wire Wire Line
 	1700 2900 1775 2900
+Text Notes 3250 5275 0    102  ~ 0
+PID
 $EndSCHEMATC

Commit message: updated: first push in Lau
Parts:
- C3, C4, C5: symbol Device:C -> incubator_bottom-rescue:C-Device
- D1, D2: symbol Diode:MBR0520LT -> incubator_bottom-rescue:MBR0520LT-Diode
- H1, H2, H3, H4, H5, H6, H7, H8: symbol Mechanical:MountingHole -> incubator_bottom-rescue:MountingHole-Mechanical
- J1, J7: symbol Connector_Generic:Conn_01x02 -> incubator_bottom-rescue:Conn_01x02-Connector_Generic
- J2: symbol Connector_Generic:Conn_02x03_Odd_Even -> incubator_bottom-rescue:Conn_02x03_Odd_Even-Connector_Generic
- J3: symbol Connector:RJ12 -> incubator_bottom-rescue:RJ12-Connector
- J4: symbol Connector_Generic:Conn_01x05 -> incubator_bottom-rescue:Conn_01x05-Connector_Generic
- J5, J6: symbol Connector:AudioJack3_SwitchTR -> incubator_bottom-rescue:AudioJack3_SwitchTR-Connector
- J8: symbol Connector_Generic:Conn_01x06 -> incubator_bottom-rescue:Conn_01x06-Connector_Generic
- Q1: symbol ZXMS6004:ZXMS6004 -> incubator_bottom-rescue:ZXMS6004-ZXMS6004
- R1, R10, R11, R13, R2, R3, R4, R5, R6, R8, R9: symbol Device:R -> incubator_bottom-rescue:R-Device
- U1: symbol Sensor_Temperature:DS18B20Z -> incubator_bottom-rescue:DS18B20Z-Sensor_Temperature
- U2: symbol Sensor_Temperature:DS18B20 -> incubator_bottom-rescue:DS18B20-Sensor_Temperature
Changed lines of the file:
@@
 $EndDescr
 $Comp
-L Sensor_Temperature:DS18B20 U2
+L incubator_bottom-rescue:DS18B20-Sensor_Temperature U2
 U 1 1 60FFAE4A
 P 10275 2875
@@
 $EndComp
 $Comp
-L Sensor_Temperature:DS18B20Z U1
+L incubator_bottom-rescue:DS18B20Z-Sensor_Temperature U1
 U 1 1 60FFDDD1
 P 6700 2750
@@
 $EndComp
 $Comp
-L Device:R R4
+L incubator_bottom-rescue:R-Device R4
 U 1 1 61013B0E
 P 7050 2550
@@
 $EndComp
 $Comp
-L power:VCC #PWR0106
+L incubator_bottom-rescue:VCC-power #PWR0106
 U 1 1 61017B63
 P 6700 2275
@@
 $EndComp
 $Comp
-L Device:R R11
+L incubator_bottom-rescue:R-Device R11
 U 1 1 61064BC7
 P 10650 2675
@@
 $EndComp
 $Comp
-L power:VCC #PWR0109
+L incubator_bottom-rescue:VCC-power #PWR0109
 U 1 1 6106C48E
 P 10275 2375
@@
 $EndComp
 $Comp
-L power:GND #PWR0110
+L incubator_bottom-rescue:GND-power #PWR0110
 U 1 1 6107013F
 P 10275 3275
@@
 	7050 2750 7000 2750
 $Comp
-L power:GND #PWR0111
+L incubator_bottom-rescue:GND-power #PWR0111
 U 1 1 61092FF6
 P 6700 3125
@@
 	6700 3050 6700 3125
 $Comp
-L power:VCC #PWR0101
+L incubator_bottom-rescue:VCC-power #PWR0101
 U 1 1 610EABF4
 P 2200 925
@@
 $EndComp
 $Comp
-L power:PWR_FLAG #FLG0101
+L incubator_bottom-rescue:PWR_FLAG-power #FLG0101
 U 1 1 610EC89D
 P 2200 775
@@
 	2200 775  2200 925
 $Comp
-L Mechanical:MountingHole H1
+L incubator_bottom-rescue:MountingHole-Mechanical H1
 U 1 1 610F54D5
 P 3325 7175
@@
 $EndComp
 $Comp
-L Mechanical:MountingHole H3
+L incubator_bottom-rescue:MountingHole-Mechanical H3
 U 1 1 610F73E9
 P 4100 7175
@@
 $EndComp
 $Comp
-L Mechanical:MountingHole H2
+L incubator_bottom-rescue:MountingHole-Mechanical H2
 U 1 1 610F770E
 P 3325 7475
@@
 $EndComp
 $Comp
-L Mechanical:MountingHole H4
+L incubator_bottom-rescue:MountingHole-Mechanical H4
 U 1 1 610F79C8
 P 4100 7475
@@
 	5050 3925 5050 3850
 $Comp
-L power:GND #PWR0102
+L incubator_bottom-rescue:GND-power #PWR0102
 U 1 1 611DACB0
 P 5050 4400
@@
 	4950 4225 5125 4225
 $Comp
-L Connector:AudioJack3_SwitchTR J5
+L incubator_bottom-rescue:AudioJack3_SwitchTR-Connector J5
 U 1 1 610A289E
 P 7850 1375
@@
 $EndComp
 $Comp
-L Device:R R6
+L incubator_bottom-rescue:R-Device R6
 U 1 1 610A3D5F
 P 7575 1050
@@
 $EndComp
 $Comp
-L Device:R R5
+L incubator_bottom-rescue:R-Device R5
 U 1 1 610A4FCA
 P 7350 1275
@@
 $EndComp
 $Comp
-L Device:R R3
+L incubator_bottom-rescue:R-Device R3
 U 1 1 610AAD8C
 P 6925 1450
@@
 $EndComp
 $Comp
-L power:VCC #PWR0103
+L incubator_bottom-rescue:VCC-power #PWR0103
 U 1 1 610BE9D4
 P 7575 800
@@
 Connection ~ 7575 1275
 $Comp
-L power:GND #PWR0104
+L incubator_bottom-rescue:GND-power #PWR0104
 U 1 1 610CEA91
 P 7575 1775
@@
 NoConn ~ 7650 1475
 $Comp
-L Mechanical:MountingHole H5
+L incubator_bottom-rescue:MountingHole-Mechanical H5
 U 1 1 6110AD0D
 P 5025 7225
@@
 $EndComp
 $Comp
-L Mechanical:MountingHole H7
+L incubator_bottom-rescue:MountingHole-Mechanical H7
 U 1 1 6110B26F
 P 5800 7225
@@
 $EndComp
 $Comp
-L Mechanical:MountingHole H6
+L incubator_bottom-rescue:MountingHole-Mechanical H6
 U 1 1 6110B9C7
 P 5025 7500
@@
 $EndComp
 $Comp
-L Mechanical:MountingHole H8
+L incubator_bottom-rescue:MountingHole-Mechanical H8
 U 1 1 6110BE5B
 P 5800 7475
@@
 $EndComp
 $Comp
-L power:+12V #PWR0105
+L incubator_bottom-rescue:+12V-power #PWR0105
 U 1 1 6111A394
 P 5050 3850
@@
 Connection ~ 5050 3925
 $Comp
-L power:+12V #PWR0108
+L incubator_bottom-rescue:+12V-power #PWR0108
 U 1 1 61121502
 P 2700 925
@@
 $EndComp
 $Comp
-L power:PWR_FLAG #FLG0102
+L incubator_bottom-rescue:PWR_FLAG-power #FLG0102
 U 1 1 611229BC
 P 2700 775
@@
 	2700 925  2700 775
 $Comp
-L Connector_Generic:Conn_01x02 J1
+L incubator_bottom-rescue:Conn_01x02-Connector_Generic J1
 U 1 1 61169294
 P 1900 5550
@@
 $EndComp
 $Comp
-L power:+12V #PWR0112
+L incubator_bottom-rescue:+12V-power #PWR0112
 U 1 1 6116C627
 P 1625 5450
@@
 	1625 5550 1700 5550
 $Comp
-L ZXMS6004:ZXMS6004 Q1
+L incubator_bottom-rescue:ZXMS6004-ZXMS6004 Q1
 U 1 1 611724A4
 P 1625 5950
@@
 	1625 5650 1700 5650
 $Comp
-L power:GND #PWR0113
+L incubator_bottom-rescue:GND-power #PWR0113
 U 1 1 6117907D
 P 1625 6450
@@
 	1875 1775 1925 1775
 $Comp
-L power:GND #PWR0107
+L incubator_bottom-rescue:GND-power #PWR0107
 U 1 1 610302A6
 P 1925 1825
@@
 MISO
 $Comp
-L Connector_Generic:Conn_02x03_Odd_Even J2
+L incubator_bottom-rescue:Conn_02x03_Odd_Even-Connector_Generic J2
 U 1 1 6104194C
 P 1575 1675
@@
 	1425 3725 1425 3675
 $Comp
-L power:VCC #PWR0114
+L incubator_bottom-rescue:VCC-power #PWR0114
 U 1 1 610EC2F5
 P 1150 3625
@@
 NoConn ~ 1700 4400
 $Comp
-L power:GND #PWR0115
+L incubator_bottom-rescue:GND-power #PWR0115
 U 1 1 610DD35E
 P 1625 4575
@@
 	1700 4000 1650 4000
 $Comp
-L Device:R R1
+L incubator_bottom-rescue:R-Device R1
 U 1 1 610DC2A0
 P 1150 3875
@@
 $EndComp
 $Comp
-L Device:R R2
+L incubator_bottom-rescue:R-Device R2
 U 1 1 610DBA03
 P 1425 3875
@@
 12V
 $Comp
-L Connector:RJ12 J3
+L incubator_bottom-rescue:RJ12-Connector J3
 U 1 1 610CF354
 P 2100 4200
@@
 $EndComp
 $Comp
-L Diode:MBR0520LT D1
+L incubator_bottom-rescue:MBR0520LT-Diode D1
 U 1 1 613041E6
 P 2250 1575
@@
 	2400 1575 2475 1575
 $Comp
-L Connector:AudioJack3_SwitchTR J6
+L incubator_bottom-rescue:AudioJack3_SwitchTR-Connector J6
 U 1 1 6148737A
 P 10075 1350
@@
 $EndComp
 $Comp
-L power:GND #PWR0116
+L incubator_bottom-rescue:GND-power #PWR0116
 U 1 1 61489A5A
 P 9800 1725
@@
 $EndComp
 $Comp
-L Device:R R10
+L incubator_bottom-rescue:R-Device R10
 U 1 1 6148A582
 P 9800 1025
@@
 $EndComp
 $Comp
-L power:VCC #PWR0117
+L incubator_bottom-rescue:VCC-power #PWR0117
 U 1 1 6148AACD
 P 9800 775
@@
 NoConn ~ 9875 1650
 $Comp
-L Device:R R9
+L incubator_bottom-rescue:R-Device R9
 U 1 1 6149E2DE
 P 9575 1250
@@
 $EndComp
 $Comp
-L Device:R R8
+L incubator_bottom-rescue:R-Device R8
 U 1 1 6149F2BA
 P 9150 1425
@@
 FAN
 $Comp
-L Connector_Generic:Conn_01x05 J4
+L incubator_bottom-rescue:Conn_01x05-Connector_Generic J4
 U 1 1 6118C3B2
 P 5325 4125
@@
 	3900 1400 3825 1400
 $Comp
-L power:GND #PWR0118
+L incubator_bottom-rescue:GND-power #PWR0118
 U 1 1 61156ECC
 P 3825 2975
@@
 NoConn ~ 8825 5000
 $Comp
-L Device:C C3
+L incubator_bottom-rescue:C-Device C3
 U 1 1 61204B1D
 P 1300 6150
@@
 Connection ~ 1300 5950
 $Comp
-L Connector_Generic:Conn_01x02 J7
+L incubator_bottom-rescue:Conn_01x02-Connector_Generic J7
 U 1 1 612511B5
 P 3925 5550
@@
 $EndComp
 $Comp
-L Device:R R13
+L incubator_bottom-rescue:R-Device R13
 U 1 1 6125F534
 P 3700 6075
@@
 $EndComp
 $Comp
-L Device:C C4
+L incubator_bottom-rescue:C-Device C4
 U 1 1 6126123D
 P 3950 6300
@@
 PID
 $Comp
-L power:GND #PWR0124
+L incubator_bottom-rescue:GND-power #PWR0124
 U 1 1 612754ED
 P 4325 6550
@@
 	4325 5550 4325 5875
 $Comp
-L power:+12V #PWR0125
+L incubator_bottom-rescue:+12V-power #PWR0125
 U 1 1 6129C970
 P 4200 5375
@@
 	4200 5450 4200 5375
 $Comp
-L Connector_Generic:Conn_01x06 J8
+L incubator_bottom-rescue:Conn_01x06-Connector_Generic J8
 U 1 1 612BD864
 P 1975 2600
@@
 ~RESET
 $Comp
-L Device:C C5
+L incubator_bottom-rescue:C-Device C5
 U 1 1 612C10B9
 P 2300 2475
@@
 $EndComp
 $Comp
-L power:GND #PWR0126
+L incubator_bottom-rescue:GND-power #PWR0126
 U 1 1 612C3665
 P 2300 2700
@@
 	1700 2600 1775 2600
 $Comp
-L Diode:MBR0520LT D2
+L incubator_bottom-rescue:MBR0520LT-Diode D2
 U 1 1 612ED8C3
 P 1475 2700
@@
 NoConn ~ 1775 2800
 $Comp
-L power:GND #PWR0127
+L incubator_bottom-rescue:GND-power #PWR0127
 U 1 1 612FF697
 P 1700 3000
