File: Kicad/incubator_bottom/incubator_bottom.sch (KiCad schematic (older format))
At the start: 42 parts, among them J1 Conn_01x02, J10 Conn_01x01, J11 Conn_01x01, J12 Conn_01x01, J2 Conn_02x03_Odd_Even, J3 RJ12, J4 Conn_01x01, J5 AudioJack3_SwitchTR, J6 AudioJack3_SwitchTR, J7 Conn_01x01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

Commit message: refactor: Power supply
Parts:
- removed J3: RJ12, Incubator:E5566-Q0LK22-L, symbol incubator_bottom-rescue:RJ12-Connector
- removed R1, R2: 10k, Resistor_SMD:R_0805_2012Metric_Pad1.20x1.40mm_HandSolder, symbol incubator_bottom-rescue:R-Device
- added C6: 0.33u, Capacitor_SMD:C_0805_2012Metric_Pad1.18x1.45mm_HandSolder, symbol incubator_bottom-rescue:C-Device
- added C7: 0.1u, Capacitor_SMD:C_0805_2012Metric_Pad1.18x1.45mm_HandSolder, symbol incubator_bottom-rescue:C-Device
- added U5: LM78M05_TO252, Package_TO_SOT_SMD:TO-252-2, symbol Regulator_Linear:LM78M05_TO252
Connections:
- net +12V: now also C6.1, U5.1 (VI)
- net GND: now also C6.2, C7.2, U5.2 (GND)
- net 5V Step-down/5V: no longer names the net of D3.2 (A)
- net 5V Step-down/5V: now also C7.1, U5.3 (VO)
- no-connect marks 8 -> 7
Other:
- note removed: "I2C\n"
- moved on the sheet: D3
Changed lines of the file:
@@
 $Descr A4 11693 8268
 encoding utf-8
-Sheet 1 3
+Sheet 1 2
 Title ""
 Date ""
@@
 C3
 Text GLabel 4750 2200 2    50   Input ~ 0
+PID
+Text GLabel 4750 2100 2    50   Input ~ 0
 FAN
-Text GLabel 4750 2100 2    50   Input ~ 0
-PID
 Text GLabel 4750 2000 2    50   Input ~ 0
 D5
@@
 Text Notes 5250 7000 0    50   ~ 0
 FAN HOLES
-$Sheet
-S 1100 4000 900  650
-U 61425B26
-F0 "5V Step-down" 50
-F1 "5V.sch" 50
-F2 "VIN" I L 1100 4200 50
-F3 "5V" O R 2000 4300 50
-F4 "GND" I L 1100 4350 50
-$EndSheet
-Text GLabel 900  4200 0    50   Input ~ 0
+Text GLabel 1050 3850 0    50   Input ~ 0
 12V
 $Comp
 L incubator_bottom-rescue:GND-power #PWR01
 U 1 1 61433F4F
-P 1000 4450
-F 0 "#PWR01" H 1000 4200 50  0001 C CNN
-F 1 "GND" H 1005 4277 50  0000 C CNN
-F 2 "" H 1000 4450 50  0001 C CNN
-F 3 "" H 1000 4450 50  0001 C CNN
-	1    1000 4450
-	1    0    0    -1
-$EndComp
-Wire Wire Line
-	1000 4450 1000 4350
-Wire Wire Line
-	1000 4350 1100 4350
-Wire Wire Line
-	1100 4200 900  4200
-Text GLabel 2500 4300 2    50   Input ~ 0
+P 1550 4450
+F 0 "#PWR01" H 1550 4200 50  0001 C CNN
+F 1 "GND" H 1555 4277 50  0000 C CNN
+F 2 "" H 1550 4450 50  0001 C CNN
+F 3 "" H 1550 4450 50  0001 C CNN
+	1    1550 4450
+	1    0    0    -1
+$EndComp
+Wire Wire Line
+	1550 4450 1550 4350
+Wire Wire Line
+	1250 3850 1150 3850
+Text GLabel 2500 3850 2    50   Input ~ 0
 VIN
 $Comp
 L incubator_bottom-rescue:MBR0520LT-Diode D3
 U 1 1 61445FAB
-P 2250 4300
-F 0 "D3" H 2250 4083 50  0000 C CNN
-F 1 "MBR0520LT" H 2250 4174 50  0000 C CNN
-F 2 "Diode_SMD:D_SOD-123" H 2250 4125 50  0001 C CNN
-F 3 "http://www.onsemi.com/pub_link/Collateral/MBR0520LT1-D.PDF" H 2250 4300 50  0001 C CNN
-	1    2250 4300
+P 2250 3850
+F 0 "D3" H 2250 3633 50  0000 C CNN
+F 1 "MBR0520LT" H 2250 3724 50  0000 C CNN
+F 2 "Diode_SMD:D_SOD-123" H 2250 3675 50  0001 C CNN
+F 3 "http://www.onsemi.com/pub_link/Collateral/MBR0520LT1-D.PDF" H 2250 3850 50  0001 C CNN
+	1    2250 3850
 	-1   0    0    1
 $EndComp
 Wire Wire Line
-	2500 4300 2400 4300
-Wire Wire Line
-	2100 4300 2000 4300
+	2500 3850 2400 3850
+Wire Wire Line
+	1950 3850 1850 3850
 $Comp
 L Connector_Generic:Conn_01x01 J7
@@
 Text Notes 650  3550 0    102  ~ 0
 5V STEP-DOWN CONVERTER
-Text Notes 1950 5375 0    150  ~ 0
-I2C\n
 Wire Notes Line
 	475  4850 5925 4850
-$Comp
-L incubator_bottom-rescue:RJ12-Connector J3
-U 1 1 610CF354
-P 2050 5900
-F 0 "J3" H 1720 5904 50  0000 R CNN
-F 1 "RJ12" H 1720 5995 50  0000 R CNN
-F 2 "Incubator:E5566-Q0LK22-L" V 2050 5925 50  0001 C CNN
-F 3 "~" V 2050 5925 50  0001 C CNN
-	1    2050 5900
-	-1   0    0    1
-$EndComp
-Text GLabel 1600 5625 1    50   Input ~ 0
-12V
-$Comp
-L incubator_bottom-rescue:R-Device R2
-U 1 1 610DBA03
-P 1375 5575
-F 0 "R2" H 1445 5621 50  0000 L CNN
-F 1 "10k" H 1445 5530 50  0000 L CNN
-F 2 "Resistor_SMD:R_0805_2012Metric_Pad1.20x1.40mm_HandSolder" V 1305 5575 50  0001 C CNN
-F 3 "~" H 1375 5575 50  0001 C CNN
-	1    1375 5575
-	1    0    0    -1
-$EndComp
-$Comp
-L incubator_bottom-rescue:R-Device R1
-U 1 1 610DC2A0
-P 1100 5575
-F 0 "R1" H 1170 5621 50  0000 L CNN
-F 1 "10k" H 1170 5530 50  0000 L CNN
-F 2 "Resistor_SMD:R_0805_2012Metric_Pad1.20x1.40mm_HandSolder" V 1030 5575 50  0001 C CNN
-F 3 "~" H 1100 5575 50  0001 C CNN
-	1    1100 5575
-	1    0    0    -1
-$EndComp
-Wire Wire Line
-	1650 5700 1600 5700
-Wire Wire Line
-	1600 5700 1600 5625
-Text GLabel 1000 5800 0    50   Input ~ 0
-SCL
-Text GLabel 1000 5900 0    50   Input ~ 0
-SDA
-$Comp
-L incubator_bottom-rescue:GND-power #PWR0115
-U 1 1 610DD35E
-P 1575 6275
-F 0 "#PWR0115" H 1575 6025 50  0001 C CNN
-F 1 "GND" H 1580 6102 50  0000 C CNN
-F 2 "" H 1575 6275 50  0001 C CNN
-F 3 "" H 1575 6275 50  0001 C CNN
-	1    1575 6275
-	1    0    0    -1
-$EndComp
-NoConn ~ 1650 6100
-Wire Wire Line
-	1650 6000 1575 6000
-Wire Wire Line
-	1575 6000 1575 6200
-Connection ~ 1575 6200
-Wire Wire Line
-	1650 6200 1575 6200
-Wire Wire Line
-	1575 6200 1575 6275
-Wire Wire Line
-	1650 5900 1100 5900
-Connection ~ 1100 5900
-Wire Wire Line
-	1650 5800 1375 5800
-Connection ~ 1375 5800
-Wire Wire Line
-	1375 5800 1375 5725
-Wire Wire Line
-	1000 5800 1375 5800
-Wire Wire Line
-	1100 5725 1100 5900
-Wire Wire Line
-	1100 5900 1000 5900
-$Comp
-L incubator_bottom-rescue:VCC-power #PWR0114
-U 1 1 610EC2F5
-P 1100 5325
-F 0 "#PWR0114" H 1100 5175 50  0001 C CNN
-F 1 "VCC" H 1115 5498 50  0000 C CNN
-F 2 "" H 1100 5325 50  0001 C CNN
-F 3 "" H 1100 5325 50  0001 C CNN
-	1    1100 5325
-	1    0    0    -1
-$EndComp
-Wire Wire Line
-	1375 5425 1375 5375
-Wire Wire Line
-	1375 5375 1100 5375
-Connection ~ 1100 5375
-Wire Wire Line
-	1100 5375 1100 5325
-Wire Wire Line
-	1100 5425 1100 5375
 Wire Notes Line
 	500  6550 5900 6550
@@
 Text Notes 4500 6500 0    50   ~ 0
 Power Resistor\n100 W 4 Ohm
+$Comp
+L Regulator_Linear:LM78M05_TO252 U5
+U 1 1 6152567E
+P 1550 3850
+F 0 "U5" H 1550 4092 50  0000 C CNN
+F 1 "LM78M05_TO252" H 1550 4001 50  0000 C CNN
+F 2 "Package_TO_SOT_SMD:TO-252-2" H 1550 4075 50  0001 C CIN
+F 3 "https://www.onsemi.com/pub/Collateral/MC78M00-D.PDF" H 1550 3800 50  0001 C CNN
+	1    1550 3850
+	1    0    0    -1
+$EndComp
+$Comp
+L incubator_bottom-rescue:C-Device C6
+U 1 1 61544A4B
+P 1150 4100
+F 0 "C6" H 1265 4146 50  0000 L CNN
+F 1 "0.33u" H 1265 4055 50  0000 L CNN
+F 2 "Capacitor_SMD:C_0805_2012Metric_Pad1.18x1.45mm_HandSolder" H 1188 3950 50  0001 C CNN
+F 3 "~" H 1150 4100 50  0001 C CNN
+	1    1150 4100
+	1    0    0    -1
+$EndComp
+$Comp
+L incubator_bottom-rescue:C-Device C7
+U 1 1 6154606C
+P 1950 4100
+F 0 "C7" H 2065 4146 50  0000 L CNN
+F 1 "0.1u" H 2065 4055 50  0000 L CNN
+F 2 "Capacitor_SMD:C_0805_2012Metric_Pad1.18x1.45mm_HandSolder" H 1988 3950 50  0001 C CNN
+F 3 "~" H 1950 4100 50  0001 C CNN
+	1    1950 4100
+	1    0    0    -1
+$EndComp
+Wire Wire Line
+	1950 3850 1950 3950
+Wire Wire Line
+	2100 3850 1950 3850
+Connection ~ 1950 3850
+Wire Wire Line
+	1150 3950 1150 3850
+Connection ~ 1150 3850
+Wire Wire Line
+	1150 3850 1050 3850
+Wire Wire Line
+	1150 4250 1150 4350
+Wire Wire Line
+	1150 4350 1550 4350
+Connection ~ 1550 4350
+Wire Wire Line
+	1550 4350 1550 4150
+Wire Wire Line
+	1950 4250 1950 4350
+Wire Wire Line
+	1950 4350 1550 4350
 $EndSCHEMATC

Commit message: refactor: final test version
Parts:
- added D4, D5: GREEN, LED_SMD:LED_0805_2012Metric_Pad1.15x1.40mm_HandSolder, symbol Device:LED
- added R1: 10k, Resistor_SMD:R_0805_2012Metric_Pad1.20x1.40mm_HandSolder, symbol Device:R
- added R2: 1k, Resistor_SMD:R_0805_2012Metric_Pad1.20x1.40mm_HandSolder, symbol Device:R
Connections:
- net +12V: now also R1.1
- net GND: now also D4.1 (K), D5.1 (K)
- net VIN: now also R2.1
- removed net ONE-WIRE: R11.2, R3.2, R4.2, R8.2, U1.4 (DQ), U2.2 (DQ)
- new net: D4.2 (A), R1.2
- new net: D5.2 (A), R2.2
- new net ONE-WIRE-1: R4.2, U1.4 (DQ)
- new net ONE-WIRE-2: R11.2, U2.2 (DQ)
- new net ONE-WIRE-3: R8.2
- new net ONE-WIRE-4: R3.2
Other:
- note added: "Power LEDS"
- moved on the sheet: C6, R11, U2
Changed lines of the file:
@@
 L incubator_bottom-rescue:DS18B20-Sensor_Temperature U2
 U 1 1 60FFAE4A
-P 10275 2875
-F 0 "U2" H 10175 2625 50  0000 R CNN
-F 1 "DS18B20" H 10175 2550 50  0000 R CNN
-F 2 "Package_TO_SOT_THT:TO-92_Inline" H 9275 2625 50  0001 C CNN
-F 3 "http://datasheets.maximintegrated.com/en/ds/DS18B20.pdf" H 10125 3125 50  0001 C CNN
-	1    10275 2875
+P 9975 2825
+F 0 "U2" H 9875 2575 50  0000 R CNN
+F 1 "DS18B20" H 9875 2500 50  0000 R CNN
+F 2 "Package_TO_SOT_THT:TO-92_Inline" H 8975 2575 50  0001 C CNN
+F 3 "http://datasheets.maximintegrated.com/en/ds/DS18B20.pdf" H 9825 3075 50  0001 C CNN
+	1    9975 2825
 	1    0    0    -1
 $EndComp
@@
 L incubator_bottom-rescue:R-Device R11
 U 1 1 61064BC7
-P 10650 2675
-F 0 "R11" H 10720 2721 50  0000 L CNN
-F 1 "4.7k" H 10720 2630 50  0000 L CNN
-F 2 "Resistor_SMD:R_0805_2012Metric_Pad1.20x1.40mm_HandSolder" V 10580 2675 50  0001 C CNN
-F 3 "~" H 10650 2675 50  0001 C CNN
-	1    10650 2675
+P 10350 2625
+F 0 "R11" H 10420 2671 50  0000 L CNN
+F 1 "4.7k" H 10420 2580 50  0000 L CNN
+F 2 "Resistor_SMD:R_0805_2012Metric_Pad1.20x1.40mm_HandSolder" V 10280 2625 50  0001 C CNN
+F 3 "~" H 10350 2625 50  0001 C CNN
+	1    10350 2625
 	1    0    0    -1
 $EndComp
@@
 L incubator_bottom-rescue:VCC-power #PWR0109
 U 1 1 6106C48E
-P 10275 2375
-F 0 "#PWR0109" H 10275 2225 50  0001 C CNN
-F 1 "VCC" H 10290 2548 50  0000 C CNN
-F 2 "" H 10275 2375 50  0001 C CNN
-F 3 "" H 10275 2375 50  0001 C CNN
-	1    10275 2375
+P 9975 2325
+F 0 "#PWR0109" H 9975 2175 50  0001 C CNN
+F 1 "VCC" H 9990 2498 50  0000 C CNN
+F 2 "" H 9975 2325 50  0001 C CNN
+F 3 "" H 9975 2325 50  0001 C CNN
+	1    9975 2325
 	1    0    0    -1
 $EndComp
@@
 L incubator_bottom-rescue:GND-power #PWR0110
 U 1 1 6107013F
-P 10275 3275
-F 0 "#PWR0110" H 10275 3025 50  0001 C CNN
-F 1 "GND" H 10280 3102 50  0000 C CNN
-F 2 "" H 10275 3275 50  0001 C CNN
-F 3 "" H 10275 3275 50  0001 C CNN
-	1    10275 3275
-	1    0    0    -1
-$EndComp
-Wire Wire Line
-	10275 3275 10275 3175
-Text GLabel 10775 2875 2    50   Input ~ 0
-ONE-WIRE
-Wire Wire Line
-	10775 2875 10650 2875
-Wire Wire Line
-	10275 2375 10275 2475
-Wire Wire Line
-	10650 2525 10650 2475
-Wire Wire Line
-	10650 2475 10275 2475
-Connection ~ 10275 2475
-Wire Wire Line
-	10275 2475 10275 2575
-Wire Wire Line
-	10650 2825 10650 2875
-Connection ~ 10650 2875
-Wire Wire Line
-	10650 2875 10575 2875
+P 9975 3225
+F 0 "#PWR0110" H 9975 2975 50  0001 C CNN
+F 1 "GND" H 9980 3052 50  0000 C CNN
+F 2 "" H 9975 3225 50  0001 C CNN
+F 3 "" H 9975 3225 50  0001 C CNN
+	1    9975 3225
+	1    0    0    -1
+$EndComp
+Wire Wire Line
+	9975 3225 9975 3125
+Text GLabel 10475 2825 2    50   Input ~ 0
+ONE-WIRE-2
+Wire Wire Line
+	10475 2825 10350 2825
+Wire Wire Line
+	9975 2325 9975 2425
+Wire Wire Line
+	10350 2475 10350 2425
+Wire Wire Line
+	10350 2425 9975 2425
+Connection ~ 9975 2425
+Wire Wire Line
+	9975 2425 9975 2525
+Wire Wire Line
+	10350 2775 10350 2825
+Connection ~ 10350 2825
+Wire Wire Line
+	10350 2825 10275 2825
 Wire Wire Line
 	6700 2275 6700 2350
@@
 	6700 2350 6700 2450
 Text GLabel 7150 2750 2    50   Input ~ 0
-ONE-WIRE
+ONE-WIRE-1
 Wire Wire Line
 	7150 2750 7050 2750
@@
 	7150 1450 7150 1275
 Text GLabel 6700 1450 0    50   Input ~ 0
-ONE-WIRE
+ONE-WIRE-4
 Wire Wire Line
 	6700 1450 6775 1450
@@
 $EndComp
 Text GLabel 8925 1425 0    50   Input ~ 0
-ONE-WIRE
+ONE-WIRE-3
 Wire Wire Line
 	9800 1175 9800 1250
@@
 FAN
 Text GLabel 4750 1025 2    50   Input ~ 0
-C0
+ONE-WIRE-4
 Text GLabel 4750 1125 2    50   Input ~ 0
-C1
+ONE-WIRE-3
 Text GLabel 4750 1225 2    50   Input ~ 0
-C2
+ONE-WIRE-2
 Text GLabel 4750 1325 2    50   Input ~ 0
-C3
+ONE-WIRE-1
 Text GLabel 4750 2200 2    50   Input ~ 0
 PID
@@
 D3
 Text GLabel 4750 1700 2    50   Input ~ 0
-ONE-WIRE
+D2
 Text GLabel 4750 1600 2    50   Input ~ 0
 TX
@@
 Text Notes 5250 7000 0    50   ~ 0
 FAN HOLES
-Text GLabel 1050 3850 0    50   Input ~ 0
+Text GLabel 1000 3850 0    50   Input ~ 0
 12V
 $Comp
@@
 	1550 4450 1550 4350
 Wire Wire Line
-	1250 3850 1150 3850
+	1250 3850 1100 3850
 Text GLabel 2500 3850 2    50   Input ~ 0
 VIN
@@
 	1    0    0    -1
 $EndComp
-NoConn ~ 4650 6300
-NoConn ~ 4650 6000
 Text Notes 4500 6500 0    50   ~ 0
 Power Resistor\n100 W 4 Ohm
@@
 L incubator_bottom-rescue:C-Device C6
 U 1 1 61544A4B
-P 1150 4100
-F 0 "C6" H 1265 4146 50  0000 L CNN
-F 1 "0.33u" H 1265 4055 50  0000 L CNN
-F 2 "Capacitor_SMD:C_0805_2012Metric_Pad1.18x1.45mm_HandSolder" H 1188 3950 50  0001 C CNN
-F 3 "~" H 1150 4100 50  0001 C CNN
-	1    1150 4100
+P 1100 4100
+F 0 "C6" H 1215 4146 50  0000 L CNN
+F 1 "0.33u" H 1215 4055 50  0000 L CNN
+F 2 "Capacitor_SMD:C_0805_2012Metric_Pad1.18x1.45mm_HandSolder" H 1138 3950 50  0001 C CNN
+F 3 "~" H 1100 4100 50  0001 C CNN
+	1    1100 4100
 	1    0    0    -1
 $EndComp
@@
 Connection ~ 1950 3850
 Wire Wire Line
-	1150 3950 1150 3850
-Connection ~ 1150 3850
-Wire Wire Line
-	1150 3850 1050 3850
-Wire Wire Line
-	1150 4250 1150 4350
-Wire Wire Line
-	1150 4350 1550 4350
+	1100 3950 1100 3850
+Connection ~ 1100 3850
+Wire Wire Line
+	1100 3850 1000 3850
+Wire Wire Line
+	1100 4250 1100 4350
+Wire Wire Line
+	1100 4350 1550 4350
 Connection ~ 1550 4350
 Wire Wire Line
@@
 Wire Wire Line
 	1950 4350 1550 4350
+NoConn ~ 4650 6000
+NoConn ~ 4650 6300
+Text Notes 700  5325 0    118  ~ 0
+Power LEDS
+$Comp
+L Device:R R?
+U 1 1 615134F4
+P 2000 5850
+AR Path="/5E0D7B92/615134F4" Ref="R?"  Part="1"
+AR Path="/5E0D7D04/615134F4" Ref="R?"  Part="1"
+AR Path="/615134F4" Ref="R2"  Part="1"
+AR Path="/5E0005EE/615134F4" Ref="R?"  Part="1"
+AR Path="/614262A1/615134F4" Ref="R?"  Part="1"
+AR Path="/61425B26/615134F4" Ref="R?"  Part="1"
+AR Path="/6150A405/615134F4" Ref="R?"  Part="1"
+F 0 "R2" V 1925 5850 50  0000 C CNN
+F 1 "1k" V 2000 5850 50  0000 C CNN
+F 2 "Resistor_SMD:R_0805_2012Metric_Pad1.20x1.40mm_HandSolder" V 1930 5850 50  0001 C CNN
+F 3 "~" H 2000 5850 50  0001 C CNN
+	1    2000 5850
+	0    1    1    0
+$EndComp
+$Comp
+L Device:LED D?
+U 1 1 61513507
+P 1500 5500
+AR Path="/6150A405/61513507" Ref="D?"  Part="1"
+AR Path="/61513507" Ref="D4"  Part="1"
+F 0 "D4" H 1500 5425 50  0000 C CNN
+F 1 "GREEN" H 1500 5600 50  0000 C CNN
+F 2 "LED_SMD:LED_0805_2012Metric_Pad1.15x1.40mm_HandSolder" H 1500 5500 50  0001 C CNN
+F 3 "~" H 1500 5500 50  0001 C CNN
+	1    1500 5500
+	1    0    0    1
+$EndComp
+Text GLabel 2300 5500 2    50   Input ~ 0
+12V
+$Comp
+L Device:R R?
+U 1 1 615134EC
+P 2000 5500
+AR Path="/5E0D7B92/615134EC" Ref="R?"  Part="1"
+AR Path="/5E0D7D04/615134EC" Ref="R?"  Part="1"
+AR Path="/615134EC" Ref="R1"  Part="1"
+AR Path="/5E0005EE/615134EC" Ref="R?"  Part="1"
+AR Path="/614262A1/615134EC" Ref="R?"  Part="1"
+AR Path="/61425B26/615134EC" Ref="R?"  Part="1"
+AR Path="/6150A405/615134EC" Ref="R?"  Part="1"
+F 0 "R1" V 1925 5500 50  0000 C CNN
+F 1 "10k" V 2000 5500 50  0000 C CNN
+F 2 "Resistor_SMD:R_0805_2012Metric_Pad1.20x1.40mm_HandSolder" V 1930 5500 50  0001 C CNN
+F 3 "~" H 2000 5500 50  0001 C CNN
+	1    2000 5500
+	0    1    1    0
+$EndComp
+Wire Wire Line
+	2300 5500 2150 5500
+Wire Wire Line
+	1850 5500 1650 5500
+$Comp
+L Device:LED D?
+U 1 1 6151350D
+P 1500 5850
+AR Path="/6150A405/6151350D" Ref="D?"  Part="1"
+AR Path="/6151350D" Ref="D5"  Part="1"
+F 0 "D5" H 1500 5775 50  0000 C CNN
+F 1 "GREEN" H 1500 5950 50  0000 C CNN
+F 2 "LED_SMD:LED_0805_2012Metric_Pad1.15x1.40mm_HandSolder" H 1500 5850 50  0001 C CNN
+F 3 "~" H 1500 5850 50  0001 C CNN
+	1    1500 5850
+	1    0    0    1
+$EndComp
+Text GLabel 2300 5850 2    50   Input ~ 0
+VIN
+Wire Wire Line
+	2300 5850 2150 5850
+Wire Wire Line
+	1850 5850 1650 5850
+$Comp
+L incubator_bottom-rescue:GND-power #PWR02
+U 1 1 61585C18
+P 1250 6000
+F 0 "#PWR02" H 1250 5750 50  0001 C CNN
+F 1 "GND" H 1255 5827 50  0000 C CNN
+F 2 "" H 1250 6000 50  0001 C CNN
+F 3 "" H 1250 6000 50  0001 C CNN
+	1    1250 6000
+	1    0    0    -1
+$EndComp
+Wire Wire Line
+	1350 5500 1250 5500
+Wire Wire Line
+	1250 5500 1250 5850
+Wire Wire Line
+	1350 5850 1250 5850
+Connection ~ 1250 5850
+Wire Wire Line
+	1250 5850 1250 6000
 $EndSCHEMATC

Commit message: feat: v1.0.1 of board
Parts:
- added D6: GREEN, LED_SMD:LED_0805_2012Metric_Pad1.15x1.40mm_HandSolder, symbol Device:LED
- added D7: RED, LED_SMD:LED_0805_2012Metric_Pad1.15x1.40mm_HandSolder, symbol Device:LED
- added R14, R15: 10k, Resistor_SMD:R_0805_2012Metric_Pad1.20x1.40mm_HandSolder, symbol Device:R
Connections:
- net GND: now also D6.1 (K), D7.1 (K); no longer C5.2
- net ~RESET: no longer J8.1 (Pin_1)
- net SCK renamed SCK|MONITORING
- net SCK|MONITORING: now also R14.2
- new net: C5.2, J8.1 (Pin_1)
- new net: D6.2 (A), R14.1
- new net: D7.2 (A), R15.1
- new net ERROR: R15.2
Other:
- moved on the sheet: C5
Changed lines of the file:
@@
 ~RESET
 Text GLabel 1275 1675 0    50   Input ~ 0
-SCK
+SCK|MONITORING
 Text GLabel 1275 1575 0    50   Input ~ 0
 MISO
@@
 ONE-WIRE-1
 Text GLabel 4750 2200 2    50   Input ~ 0
+D7
+Text GLabel 4750 2100 2    50   Input ~ 0
 PID
-Text GLabel 4750 2100 2    50   Input ~ 0
+Text GLabel 4750 2000 2    50   Input ~ 0
 FAN
-Text GLabel 4750 2000 2    50   Input ~ 0
-D5
 Text GLabel 4750 1900 2    50   Input ~ 0
 D4
@@
 Text GLabel 4750 2750 2    50   Input ~ 0
 SDA
-Text GLabel 4750 2575 2    50   Input ~ 0
-SCK
-Text GLabel 4750 2475 2    50   Input ~ 0
+Text GLabel 4750 2550 2    50   Input ~ 0
+SCK|MONITORING
+Text GLabel 4750 2450 2    50   Input ~ 0
 MISO
-Text GLabel 4750 2375 2    50   Input ~ 0
+Text GLabel 4750 2350 2    50   Input ~ 0
 MOSI
 Text GLabel 3825 1400 0    50   Input ~ 0
@@
 F17 "~RESET" I L 3900 1400 50
 F18 "VIN" I L 3900 1300 50
-F19 "MOSI" I R 4675 2375 50
-F20 "MISO" I R 4675 2475 50
-F21 "SCK" I R 4675 2575 50
+F19 "MOSI" I R 4675 2350 50
+F20 "MISO" I R 4675 2450 50
+F21 "SCK" I R 4675 2550 50
+F22 "ERROR" I R 4675 2650 50
 $EndSheet
 Wire Wire Line
@@
 Wire Wire Line
 	4750 2200 4675 2200
-Wire Wire Line
-	4675 2575 4750 2575
-Wire Wire Line
-	4750 2475 4675 2475
-Wire Wire Line
-	4675 2375 4750 2375
 Text GLabel 3825 1300 0    50   Input ~ 0
 VIN
@@
 	1    0    0    -1
 $EndComp
-Text GLabel 2425 2250 2    50   Input ~ 0
+Text GLabel 2525 2250 2    50   Input ~ 0
 ~RESET
 $Comp
 L incubator_bottom-rescue:C-Device C5
 U 1 1 612C10B9
-P 2300 2475
-F 0 "C5" H 2415 2521 50  0000 L CNN
-F 1 "100n" H 2415 2430 50  0000 L CNN
-F 2 "Capacitor_SMD:C_0805_2012Metric_Pad1.18x1.45mm_HandSolder" H 2338 2325 50  0001 C CNN
-F 3 "~" H 2300 2475 50  0001 C CNN
-	1    2300 2475
-	1    0    0    -1
-$EndComp
-$Comp
-L incubator_bottom-rescue:GND-power #PWR0126
-U 1 1 612C3665
-P 2300 2700
-F 0 "#PWR0126" H 2300 2450 50  0001 C CNN
-F 1 "GND" H 2305 2527 50  0000 C CNN
-F 2 "" H 2300 2700 50  0001 C CNN
-F 3 "" H 2300 2700 50  0001 C CNN
-	1    2300 2700
-	1    0    0    -1
-$EndComp
-Wire Wire Line
-	2300 2700 2300 2625
-Wire Wire Line
-	2425 2250 2300 2250
-Wire Wire Line
-	2300 2250 2300 2325
+P 2275 2250
+F 0 "C5" H 2390 2296 50  0000 L CNN
+F 1 "100n" H 2390 2205 50  0000 L CNN
+F 2 "Capacitor_SMD:C_0805_2012Metric_Pad1.18x1.45mm_HandSolder" H 2313 2100 50  0001 C CNN
+F 3 "~" H 2275 2250 50  0001 C CNN
+	1    2275 2250
+	0    1    1    0
+$EndComp
 Wire Wire Line
 	1775 2400 1700 2400
 Wire Wire Line
 	1700 2400 1700 2250
-Wire Wire Line
-	1700 2250 2300 2250
-Connection ~ 2300 2250
 Text GLabel 4750 1500 2    50   Input ~ 0
 RX
@@
 Wire Wire Line
 	1250 5850 1250 6000
+Wire Wire Line
+	1700 2250 2125 2250
+Wire Wire Line
+	2425 2250 2525 2250
+$Comp
+L Device:R R?
+U 1 1 61973D5B
+P 1500 6725
+AR Path="/5E0D7B92/61973D5B" Ref="R?"  Part="1"
+AR Path="/5E0D7D04/61973D5B" Ref="R?"  Part="1"
+AR Path="/61973D5B" Ref="R14"  Part="1"
+AR Path="/5E0005EE/61973D5B" Ref="R?"  Part="1"
+AR Path="/614262A1/61973D5B" Ref="R?"  Part="1"
+AR Path="/61425B26/61973D5B" Ref="R?"  Part="1"
+AR Path="/6150A405/61973D5B" Ref="R?"  Part="1"
+F 0 "R14" V 1425 6725 50  0000 C CNN
+F 1 "10k" V 1500 6725 50  0000 C CNN
+F 2 "Resistor_SMD:R_0805_2012Metric_Pad1.20x1.40mm_HandSolder" V 1430 6725 50  0001 C CNN
+F 3 "~" H 1500 6725 50  0001 C CNN
+	1    1500 6725
+	0    1    1    0
+$EndComp
+$Comp
+L Device:LED D?
+U 1 1 61975EC7
+P 1900 6725
+AR Path="/6150A405/61975EC7" Ref="D?"  Part="1"
+AR Path="/61975EC7" Ref="D6"  Part="1"
+F 0 "D6" H 1900 6650 50  0000 C CNN
+F 1 "GREEN" H 1900 6825 50  0000 C CNN
+F 2 "LED_SMD:LED_0805_2012Metric_Pad1.15x1.40mm_HandSolder" H 1900 6725 50  0001 C CNN
+F 3 "~" H 1900 6725 50  0001 C CNN
+	1    1900 6725
+	-1   0    0    -1
+$EndComp
+Text GLabel 1250 6725 0    50   Input ~ 0
+SCK|MONITORING
+Wire Wire Line
+	1250 6725 1350 6725
+Wire Wire Line
+	1650 6725 1750 6725
+$Comp
+L incubator_bottom-rescue:GND-power #PWR0114
+U 1 1 61986C2C
+P 2200 7125
+F 0 "#PWR0114" H 2200 6875 50  0001 C CNN
+F 1 "GND" H 2205 6952 50  0000 C CNN
+F 2 "" H 2200 7125 50  0001 C CNN
+F 3 "" H 2200 7125 50  0001 C CNN
+	1    2200 7125
+	1    0    0    -1
+$EndComp
+$Comp
+L Device:R R?
+U 1 1 61994E89
+P 1500 7025
+AR Path="/5E0D7B92/61994E89" Ref="R?"  Part="1"
+AR Path="/5E0D7D04/61994E89" Ref="R?"  Part="1"
+AR Path="/61994E89" Ref="R15"  Part="1"
+AR Path="/5E0005EE/61994E89" Ref="R?"  Part="1"
+AR Path="/614262A1/61994E89" Ref="R?"  Part="1"
+AR Path="/61425B26/61994E89" Ref="R?"  Part="1"
+AR Path="/6150A405/61994E89" Ref="R?"  Part="1"
+F 0 "R15" V 1425 7025 50  0000 C CNN
+F 1 "10k" V 1500 7025 50  0000 C CNN
+F 2 "Resistor_SMD:R_0805_2012Metric_Pad1.20x1.40mm_HandSolder" V 1430 7025 50  0001 C CNN
+F 3 "~" H 1500 7025 50  0001 C CNN
+	1    1500 7025
+	0    1    1    0
+$EndComp
+$Comp
+L Device:LED D?
+U 1 1 619952CE
+P 1925 7025
+AR Path="/6150A405/619952CE" Ref="D?"  Part="1"
+AR Path="/619952CE" Ref="D7"  Part="1"
+F 0 "D7" H 1925 6950 50  0000 C CNN
+F 1 "RED" H 1925 7125 50  0000 C CNN
+F 2 "LED_SMD:LED_0805_2012Metric_Pad1.15x1.40mm_HandSolder" H 1925 7025 50  0001 C CNN
+F 3 "~" H 1925 7025 50  0001 C CNN
+	1    1925 7025
+	-1   0    0    -1
+$EndComp
+Text GLabel 1225 7025 0    50   Input ~ 0
+ERROR
+Text GLabel 4750 2650 2    50   Input ~ 0
+ERROR
+Wire Wire Line
+	4675 2350 4750 2350
+Wire Wire Line
+	4750 2450 4675 2450
+Wire Wire Line
+	4675 2550 4750 2550
+Wire Wire Line
+	4750 2650 4675 2650
+Wire Wire Line
+	1225 7025 1350 7025
+Wire Wire Line
+	1650 7025 1775 7025
+Wire Wire Line
+	2075 7025 2200 7025
+Wire Wire Line
+	2200 7025 2200 7125
+Wire Wire Line
+	2050 6725 2200 6725
+Wire Wire Line
+	2200 6725 2200 7025
+Connection ~ 2200 7025
 $EndSCHEMATC
