File: Kicad/incubator_bottom/incubator_bottom.sch (KiCad schematic (older format))
At the start: 50 parts, among them J1 Conn_01x02, J10 Conn_01x01, J11 Conn_01x01, J12 Conn_01x01, J2 Conn_02x03_Odd_Even, J4 Conn_01x01, J5 AudioJack3_SwitchTR, J6 AudioJack3_SwitchTR, J7 Conn_01x01, J8 Conn_01x06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

Commit message: fix: change diameter of holes and put logo
Parts:
- H1, H2, H3, H4: footprint MountingHole:MountingHole_3.2mm_M3 -> MountingHole:MountingHole_4.3mm_M4
Changed lines of the file:
@@
 F 0 "H1" H 3425 7221 50  0000 L CNN
 F 1 "MountingHole" H 3425 7130 50  0000 L CNN
-F 2 "MountingHole:MountingHole_3.2mm_M3" H 3325 7175 50  0001 C CNN
+F 2 "MountingHole:MountingHole_4.3mm_M4" H 3325 7175 50  0001 C CNN
 F 3 "~" H 3325 7175 50  0001 C CNN
 	1    3325 7175
@@
 F 0 "H3" H 4200 7221 50  0000 L CNN
 F 1 "MountingHole" H 4200 7130 50  0000 L CNN
-F 2 "MountingHole:MountingHole_3.2mm_M3" H 4100 7175 50  0001 C CNN
+F 2 "MountingHole:MountingHole_4.3mm_M4" H 4100 7175 50  0001 C CNN
 F 3 "~" H 4100 7175 50  0001 C CNN
 	1    4100 7175
@@
 F 0 "H2" H 3425 7521 50  0000 L CNN
 F 1 "MountingHole" H 3425 7430 50  0000 L CNN
-F 2 "MountingHole:MountingHole_3.2mm_M3" H 3325 7475 50  0001 C CNN
+F 2 "MountingHole:MountingHole_4.3mm_M4" H 3325 7475 50  0001 C CNN
 F 3 "~" H 3325 7475 50  0001 C CNN
 	1    3325 7475
@@
 F 0 "H4" H 4200 7521 50  0000 L CNN
 F 1 "MountingHole" H 4200 7430 50  0000 L CNN
-F 2 "MountingHole:MountingHole_3.2mm_M3" H 4100 7475 50  0001 C CNN
+F 2 "MountingHole:MountingHole_4.3mm_M4" H 4100 7475 50  0001 C CNN
 F 3 "~" H 4100 7475 50  0001 C CNN
 	1    4100 7475

Commit message: fix: version 1.0.2 of the PCB change size holes M4 -> M3 and changes their position
Parts:
- H1, H2, H3, H4: footprint MountingHole:MountingHole_4.3mm_M4 -> MountingHole:MountingHole_3.2mm_M3
Changed lines of the file:
@@
 F 0 "H1" H 3425 7221 50  0000 L CNN
 F 1 "MountingHole" H 3425 7130 50  0000 L CNN
-F 2 "MountingHole:MountingHole_4.3mm_M4" H 3325 7175 50  0001 C CNN
+F 2 "MountingHole:MountingHole_3.2mm_M3" H 3325 7175 50  0001 C CNN
 F 3 "~" H 3325 7175 50  0001 C CNN
 	1    3325 7175
@@
 F 0 "H3" H 4200 7221 50  0000 L CNN
 F 1 "MountingHole" H 4200 7130 50  0000 L CNN
-F 2 "MountingHole:MountingHole_4.3mm_M4" H 4100 7175 50  0001 C CNN
+F 2 "MountingHole:MountingHole_3.2mm_M3" H 4100 7175 50  0001 C CNN
 F 3 "~" H 4100 7175 50  0001 C CNN
 	1    4100 7175
@@
 F 0 "H2" H 3425 7521 50  0000 L CNN
 F 1 "MountingHole" H 3425 7430 50  0000 L CNN
-F 2 "MountingHole:MountingHole_4.3mm_M4" H 3325 7475 50  0001 C CNN
+F 2 "MountingHole:MountingHole_3.2mm_M3" H 3325 7475 50  0001 C CNN
 F 3 "~" H 3325 7475 50  0001 C CNN
 	1    3325 7475
@@
 F 0 "H4" H 4200 7521 50  0000 L CNN
 F 1 "MountingHole" H 4200 7430 50  0000 L CNN
-F 2 "MountingHole:MountingHole_4.3mm_M4" H 4100 7475 50  0001 C CNN
+F 2 "MountingHole:MountingHole_3.2mm_M3" H 4100 7475 50  0001 C CNN
 F 3 "~" H 4100 7475 50  0001 C CNN
 	1    4100 7475
