File: Kicad/incubator_bottom/incubator_bottom.kicad_pcb (KiCad board)
At the start: 2 copper layers, 100.1 x 73.7 mm, 57 parts, among them J1 Conn_01x02, J10 Conn_01x01, J11 Conn_01x01, J12 Conn_01x01, J2 Conn_02x03_Odd_Even, J4 Conn_01x01, J5 AudioJack3_SwitchTR, J6 AudioJack3_SwitchTR, J7 Conn_01x01, J8 Conn_01x06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

Commit message: refactor: Power supply
Parts:
- removed C8, C9: 22µF, Capacitor_SMD:C_0805_2012Metric_Pad1.18x1.45mm_HandSolder
- removed D4: MBR0520LT, Diode_SMD:D_SOD-123
- removed D5, D6: GREEN, LED_SMD:LED_0805_2012Metric_Pad1.15x1.40mm_HandSolder
- removed L1: 4.7µH, Inductor_SMD:L_Taiyo-Yuden_NR-40xx_HandSoldering
- removed R14: 9.64k, Resistor_SMD:R_0805_2012Metric_Pad1.20x1.40mm_HandSolder
- removed R15: 49.9k, Resistor_SMD:R_0805_2012Metric_Pad1.20x1.40mm_HandSolder
- removed R16: 10k, Resistor_SMD:R_0805_2012Metric_Pad1.20x1.40mm_HandSolder
- removed R17: 1k, Resistor_SMD:R_0805_2012Metric_Pad1.20x1.40mm_HandSolder
- removed U4: ACT4088, Package_TO_SOT_SMD:SOT-23-6_Handsoldering
- added U5: LM78M05_TO252, Package_TO_SOT_SMD:TO-252-2, F.Cu at (157.9, 67.6)
- C6: value 10µF -> 0.33u
- C7: value 22nF -> 0.1u
- moved U1 55.3 mm to (97.8, 109.3)
- moved R4 55.3 mm to (92.3, 110.1)
- moved C7 18.3 mm to (161.3, 74.7), turned to 0 degrees
- moved D3 9.08 mm to (160.0, 78.6), turned to 90 degrees
- moved C6 7.70 mm to (154.4, 74.8), turned to 180 degrees
- moved D2 3.30 mm to (158.8, 113.0), turned to 180 degrees
- moved C3 2.16 mm to (152.1, 120.4)
- moved J1 2.16 mm to (139.8, 118.4)
- moved Q1 2.16 mm to (148.5, 118.4)
- moved Q2 0.89 mm to (96.0, 118.7)
- moved C5 0.36 mm to (149.5, 98.0)
Connections:
- C7 pad 2: Net-(C7-Pad2) -> GND
- D3 pad 2: /5V Step-down/5V -> Net-(C7-Pad1)
- U3 pad 10: PID -> FAN
- U3 pad 11: FAN -> PID
Routing:
- net ONE-WIRE: track 41.4 -> 207.9 mm
- net VIN: track 117.5 -> 238.3 mm, vias 4 -> 7
- net 12V: track 112.6 -> 148.4 mm, vias 57 -> 59
- net FAN: track 72.7 -> 39.5 mm
- net /5V Step-down/5V: track 25.3 -> 0.00 mm
- net SDA: track 33.9 -> 57.2 mm, vias 1 -> 2
- net SCL: track 32.0 -> 49.2 mm, vias 1 -> 2
- net Net-(C7-Pad2): track 11.2 -> 0.00 mm
- net Net-(R14-Pad2): track 4.93 -> 0.00 mm
- net PID: track 126.0 -> 122.3 mm
- net Net-(D5-Pad2): track 2.69 -> 0.00 mm
- net Net-(D6-Pad2): track 2.43 -> 0.00 mm
- net GND: track 10.9 -> 9.28 mm, vias 12 -> 19
- net RX: track 16.2 -> 16.8 mm
Other:
- board text added: "GND"
- board text added: "SCL"
- board text added: "SDA"
- board text added: "VCC"
- board text added: "⏚"

Commit message: refactor: Power supply pads
Parts:
- J10, J11, J4, J9: moved to B.Cu
- moved J7 2.29 mm to (126.7, 121.8)
- moved J12 2.03 mm to (111.4, 121.5)
- moved R7 0.38 mm to (117.9, 84.2)
Routing:
- net 12V: track 148.4 -> 184.2 mm, vias 59 -> 86
- net SDA: track 57.2 -> 52.0 mm, vias 2 -> 3
- net SCL: track 49.2 -> 44.2 mm, vias 2 -> 3
- net FAN: track 39.5 -> 36.1 mm
- net ONE-WIRE: track 207.9 -> 206.4 mm
- net PID: track 122.3 -> 121.6 mm
- net VIN: track 238.3 -> 238.9 mm
- net GND: vias 19 -> 23
Other:
- outline, holes or cut-outs redrawn
- board text added: "Incubator V 1.0"

Commit message: refactor: final test version
Parts:
- added D4: GREEN, LED_SMD:LED_0805_2012Metric_Pad1.15x1.40mm_HandSolder, F.Cu at (83.2, -60.6)
- added D5: GREEN, LED_SMD:LED_0805_2012Metric_Pad1.15x1.40mm_HandSolder, F.Cu at (96.6, -60.6)
- added R1: 10k, Resistor_SMD:R_0805_2012Metric_Pad1.20x1.40mm_HandSolder, F.Cu at (83.2, -56.4)
- added R2: 1k, Resistor_SMD:R_0805_2012Metric_Pad1.20x1.40mm_HandSolder, F.Cu at (96.6, -56.3)
- added logoHackuarium: , Incubator:logoHackuarium, F.Cu at (0.00, -18.8)
- moved C5 146.1 mm to (81.7, -31.4)
- moved C1 144.4 mm to (91.5, -22.0)
- moved C2 144.4 mm to (91.5, -24.6)
- moved C3 144.4 mm to (83.9, -6.86)
- moved C4 144.4 mm to (17.3, -9.12)
- moved C6 144.4 mm to (86.2, -52.5)
- moved C7 144.4 mm to (93.1, -52.6)
- moved D1 144.4 mm to (89.3, -40.6)
- moved D2 144.4 mm to (90.6, -14.2)
- moved D3 144.4 mm to (91.8, -48.6)
- moved H5 144.4 mm to (31.2, -65.7)
- moved H6 144.4 mm to (31.2, -28.3)
- moved H7 144.4 mm to (71.3, -65.7)
- moved H8 144.4 mm to (71.3, -28.3)
- moved J1 144.4 mm to (71.6, -8.89)
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Connections:
- R11 pad 2: ONE-WIRE -> ONE-WIRE-2
- R3 pad 2: ONE-WIRE -> ONE-WIRE-4
- R4 pad 2: ONE-WIRE -> ONE-WIRE-1
- R8 pad 2: ONE-WIRE -> ONE-WIRE-3
- U1 pad 4: ONE-WIRE -> ONE-WIRE-1
- U2 pad 2: ONE-WIRE -> ONE-WIRE-2
- U3 pad 23: C0 -> ONE-WIRE-4
- U3 pad 24: C1 -> ONE-WIRE-3
- U3 pad 25: C2 -> ONE-WIRE-2
- U3 pad 26: C3 -> ONE-WIRE-1
- U3 pad 32: ONE-WIRE -> D2
Routing:
- net ONE-WIRE: track 206.4 -> 0.00 mm, vias 2 -> 0
- net ONE-WIRE-4: track 0.00 -> 143.8 mm, vias 0 -> 2
- net ONE-WIRE-3: track 0.00 -> 126.6 mm, vias 0 -> 2
- net ONE-WIRE-2: track 0.00 -> 118.2 mm, vias 0 -> 4
- net ONE-WIRE-1: track 0.00 -> 88.6 mm, vias 0 -> 4
- net VIN: track 238.9 -> 254.1 mm
- net 12V: track 184.2 -> 190.2 mm
- net Net-(D5-Pad2): track 0.00 -> 2.28 mm
- net Net-(D4-Pad2): track 0.00 -> 2.19 mm
- net GND: track 9.28 -> 9.93 mm, vias 23 -> 45
Other:
- board size 100.1 x 73.7 mm -> 99.9 x 73.7 mm
- board text added: "5V"
- board text added: "Incubator V 1.0.0"
- board text removed: "Incubator V 1.0"
